Commit message: Fix right-hand URDF assembly (codex round-6 BLOCKING)
- build_iiwa14_right_sharpa_urdf.py: replaced tail-chop with surgical
  removal of every <link name='left_*'> block and every <joint> whose
  parent or child is a left_* link.  This preserves the
  iiwa14_link_ee → sharpa_mount joint that sits at the very end of the
  source URDF and was being silently dropped, leaving sharpa_mount
  orphaned from the arm.
- Mesh copy now filters by the right_sharpa_meshes/ prefix only, so
  iiwa14 STL refs no longer trigger false-positive missing warnings.
- Regenerated assets/urdf/.../iiwa14_right_sharpa_adjusted_restricted.urdf
  (45 links, 44 joints, 29 movable, 0 orphans, 0 left leftovers); the
  full chain is now reachable from iiwa14_link_0.

File: assets/urdf/kuka_sharpa_description/iiwa14_right_sharpa_adjusted_restricted.urdf (robot description, URDF)
Before this commit: robot kuka_sharpa, 45 links, 43 joints
Joints:
- added joint iiwa14_sharpa: type fixed, parent iiwa14_link_ee, child sharpa_mount, origin xyz=0.00 0 0 rpy=0 0 0.261799
